Commit message: Separate the "table" model for collision detection

File: ur5_rl/resources/models/models/ur5_env.urdf (robot description, URDF)
Before this commit: robot ur5e_robot, 42 links, 41 joints
Links:
- removed link aruco
- removed link table
- link base: mass None -> 0.0
- link base_cylinder: mass None -> 0.0
- link base_link: mass None -> 0.0
- link camera_bottom_screw_frame: mass None -> 0.0
- link camera_color_frame: mass None -> 0.0
- link camera_color_optical_frame: mass None -> 0.0
- link camera_depth_frame: mass None -> 0.0
- link camera_depth_optical_frame: mass None -> 0.0
- link camera_left_ir_frame: mass None -> 0.0
- link camera_left_ir_optical_frame: mass None -> 0.0
- link camera_right_ir_frame: mass None -> 0.0
- link camera_right_ir_optical_frame: mass None -> 0.0
- link ee_link: mass None -> 0.0
- link flange: mass None -> 0.0
- link ground: mass None -> 0.0
- link robotiq_tool0: mass None -> 1.3
- link tool0: mass None -> 0.0
- link world: mass None -> 0.0
Joints:
- removed joint aruco_table_joint
- removed joint world_table_joint

Commit message: Delete ground plane

File: ur5_rl/resources/models/models/ur5_env.urdf (robot description, URDF)
Before this commit: robot ur5e_robot, 40 links, 39 joints
Links:
- removed link ground
Joints:
- removed joint world_ground_joint

Commit message: Rotate last flange of the fingers

File: ur5_rl/resources/models/models/ur5_env.urdf (robot description, URDF)
Before this commit: robot ur5e_robot, 39 links, 38 joints
Joints:
- joint robotiq_finger_1_joint_3: origin xyz=0.039 0 0 rpy=0 0 0 -> xyz=0.039 0 0 rpy=0 0 -0.6
- joint robotiq_finger_2_joint_3: origin xyz=0.039 0 0 rpy=0 0 0 -> xyz=0.039 0 0 rpy=0 0 -0.6
- joint robotiq_finger_middle_joint_3: origin xyz=0.039 0 0 rpy=0 0 0 -> xyz=0.039 0 0 rpy=0 0 -0.6

Commit message: Collision on the inner finger parts

File: ur5_rl/resources/models/models/ur5_env.urdf (robot description, URDF)
Before this commit: robot ur5e_robot, 39 links, 38 joints
Links:
- added link contact1, mass 0.0; collision box size=0.008 0.1 0.027; visual box size=0.008 0.1 0.027
- added link contact2, mass 0.0; collision box size=0.008 0.1 0.027; visual box size=0.008 0.1 0.027
- added link contact3, mass 0.0; collision box size=0.008 0.1 0.027; visual box size=0.008 0.1 0.027
Joints:
- added joint contact1_finger1: type fixed, parent robotiq_finger_middle_link_3, child contact1, origin xyz=-0.018 -0.0075 0.0 rpy=0.0 0.0 2.21
- added joint contact2_finger1: type fixed, parent robotiq_finger_1_link_3, child contact2, origin xyz=-0.018 -0.0075 0.0 rpy=0.0 0.0 2.21
- added joint contact3_finger1: type fixed, parent robotiq_finger_2_link_3, child contact3, origin xyz=-0.018 -0.0075 0.0 rpy=0.0 0.0 2.21

Commit message: Add third camera

File: ur5_rl/resources/models/models/ur5_env.urdf (robot description, URDF)
Before this commit: robot ur5e_robot, 42 links, 41 joints
Joints:
- joint camera_link_joint: origin xyz=0 0.0175 0.0125 rpy=0 0 0 -> xyz=0 0.0175 0.0125 rpy=0 -0.4 0
