Commit message: Two arucos for RANSAC essential matrix estimation

File: ur5_rl/resources/models/models/table.urdf (robot description, URDF)
Before this commit: robot ur5e_robot, 2 links, 1 joints
Links:
- added link aruco_2, mass 0.0; visual mesh filename=./untitled.obj scale=0.1 0.1 0.1
Joints:
- added joint aruco2_table_joint: type fixed, parent table, child aruco_2, origin xyz=0.405 -0.01 0.055 rpy=0.0 0.0 -1.57

Commit message: Added background

File: ur5_rl/resources/models/models/table.urdf (robot description, URDF)
Before this commit: robot ur5e_robot, 3 links, 2 joints
Links:
- added link background, mass 0.0; visual mesh filename=./background.obj scale=2 2 2
Joints:
- added joint background_table_joint: type fixed, parent table, child background, origin xyz=1.3 -0.6 0.3 rpy=3.1415 3.1415 0.0

Commit message: Put the arucos more farther from the camera

File: ur5_rl/resources/models/models/table.urdf (robot description, URDF)
Before this commit: robot ur5e_robot, 4 links, 3 joints
Joints:
- joint aruco2_table_joint: origin xyz=0.405 -0.01 0.055 rpy=0.0 0.0 -1.57 -> xyz=0.455 -0.01 0.055 rpy=0.0 0.0 -1.57
- joint aruco_table_joint: origin xyz=0.30 -0.01 0.055 rpy=0.0 0.0 -1.57 -> xyz=0.35 -0.01 0.055 rpy=0.0 0.0 -1.57

Commit message: One aruco. Background to fit in image

File: ur5_rl/resources/models/models/table.urdf (robot description, URDF)
Before this commit: robot ur5e_robot, 4 links, 3 joints
Links:
- removed link aruco_2
Joints:
- removed joint aruco2_table_joint
- joint background_table_joint: origin xyz=1.3 -0.6 0.3 rpy=3.1415 3.1415 0.0 -> xyz=1.1 -0.6 0.3 rpy=3.1415 3.1415 0.0

Commit message: DQ_5.0.1

File: ur5_rl/resources/models/models/table.urdf (robot description, URDF)
Before this commit: robot ur5e_robot, 3 links, 2 joints
Links:
- removed link aruco
Joints:
- removed joint aruco_table_joint

File: ur5_rl/resources/models/models/ur5_env.urdf (robot description, URDF)
Before this commit: robot ur5e_robot, 42 links, 41 joints
Links:
- removed link contact1
- removed link contact2
- removed link contact3
Joints:
- removed joint contact1_finger1
- removed joint contact2_finger1
- removed joint contact3_finger1

Commit message: Try to get the 5.0 model

File: ur5_rl/resources/models/models/table.urdf (robot description, URDF)
Before this commit: robot ur5e_robot, 2 links, 1 joints
Links:
- added link aruco, mass 0.0; visual mesh filename=./untitled.obj scale=0.1 0.1 0.1
Joints:
- added joint aruco_table_joint: type fixed, parent table, child aruco, origin xyz=0.35 -0.01 0.055 rpy=0.0 0.0 -1.57

File: ur5_rl/resources/models/models/ur5_env.urdf (robot description, URDF)
Before this commit: robot ur5e_robot, 39 links, 38 joints
Links:
- added link contact1, mass 0.0; collision box size=0.008 0.1 0.027; visual box size=0.008 0.1 0.027
- added link contact2, mass 0.0; collision box size=0.008 0.1 0.027; visual box size=0.008 0.1 0.027
- added link contact3, mass 0.0; collision box size=0.008 0.1 0.027; visual box size=0.008 0.1 0.027
Joints:
- added joint contact1_finger1: type fixed, parent robotiq_finger_middle_link_3, child contact1, origin xyz=-0.018 -0.0075 0.0 rpy=0.0 0.0 2.21
- added joint contact2_finger1: type fixed, parent robotiq_finger_1_link_3, child contact2, origin xyz=-0.018 -0.0075 0.0 rpy=0.0 0.0 2.21
- added joint contact3_finger1: type fixed, parent robotiq_finger_2_link_3, child contact3, origin xyz=-0.018 -0.0075 0.0 rpy=0.0 0.0 2.21

Commit message: DQ_5.2_aux

File: ur5_rl/resources/models/models/table.urdf (robot description, URDF)
Before this commit: robot ur5e_robot, 3 links, 2 joints
Links:
- removed link aruco
Joints:
- removed joint aruco_table_joint

Commit message: DQ_6.0_MultipleObjects

File: ur5_rl/resources/models/models/table.urdf (robot description, URDF)
Before this commit: robot ur5e_robot, 2 links, 1 joints
Links:
- added link background_2, mass 0.0; visual mesh filename=./background_2.obj scale=2 2 2
Joints:
- added joint background2_table_joint: type fixed, parent table, child background_2, origin xyz=0.0 -0.5 -0.2 rpy=3.1415 -1.57 -0.08
