Commit message: Dummy link to test collision (test)

File: ur5_rl/resources/models/pybullet_URDF_objects/002_master_chef_can/model.urdf (robot description, URDF)
Before this commit: robot model.urdf, 1 links, 0 joints
Links:
- added link dummy, mass 0
Joints:
- added joint dummyJoint: type fixed, parent baseLink, child dummy, origin xyz=0.0 0.0 0.0 rpy=0.0 0.0 0.0

Commit message: Grasping tests

File: ur5_rl/resources/models/pybullet_URDF_objects/002_master_chef_can/model.urdf (robot description, URDF)
Before this commit: robot model.urdf, 2 links, 1 joints
Links:
- link baseLink: mass 50 -> 1
