Commit message: Object Spawning in Gazebo

File: ros_ws/src/ur5_rl/urdf/002_master_chef_can/model.urdf (robot description, URDF)
Before this commit: robot model.urdf, 2 links, 1 joints
Links:
- removed link baseLink
- added link objectLink, mass 0.2; collision mesh filename=/daniel/Desktop/ur5-rl/ros_ws/src/ur5_rl/urdf/002_master_ch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 scale=1 1 1; visual mesh filename=/daniel/Desktop/ur5-rl/ros_ws/src/ur5_rl/urdf/002_master_ch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 scale=1 1 1
Joints:
- joint dummyJoint: parent baseLink -> objectLink
