Commit message: Model test for Gazebo

File: ros_ws/src/experiment_settings/urdf/ur5e_sim.xacro (robot description, xacro)
@@ -61,13 +61,11 @@
   <!-- camera body, with origin at bottom screw mount -->
   <link name="camera_link">
-    <visual>
+    <!-- <visual>
       <origin rpy="1.5707963267948966 0 1.5707963267948966" xyz="0.0149 -0.0175 0"/>
       <geometry>
-        <!-- <box size="${d435_cam_width} ${d435_cam_height} ${d435_cam_depth}"/> -->
         <mesh filename="package://experiment_settings/meshes/d435_sim.dae"/>
-        <!--<mesh filename="package://realsense2_description/meshes/d435/d435.dae" />-->
       </geometry>
       <material name="camera_aluminum"/>
-    </visual>
+    </visual> -->
     <collision>
       <origin rpy="0 0 0" xyz="0 -0.0175 0"/>
@@ -84,13 +82,11 @@
   </link>
   <link name="camera_link_frontal">
-    <visual>
+    <!-- <visual>
       <origin rpy="1.5707963267948966 0 1.5707963267948966" xyz="0.0149 -0.0175 0"/>
       <geometry>
-        <!-- <box size="${d435_cam_width} ${d435_cam_height} ${d435_cam_depth}"/> -->
         <mesh filename="package://experiment_settings/meshes/d435_sim.dae"/>
-        <!--<mesh filename="package://realsense2_description/meshes/d435/d435.dae" />-->
       </geometry>
       <material name="camera_aluminum"/>
-    </visual>
+    </visual> -->
     <collision>
       <origin rpy="0 0 0" xyz="0 -0.0175 0"/>
@@ -107,13 +103,11 @@
   </link>
   <link name="camera_link_side">
-    <visual>
+    <!-- <visual>
       <origin rpy="1.5707963267948966 0 1.5707963267948966" xyz="0.0149 -0.0175 0"/>
       <geometry>
-        <!-- <box size="${d435_cam_width} ${d435_cam_height} ${d435_cam_depth}"/> -->
         <mesh filename="package://experiment_settings/meshes/d435_sim.dae"/>
-        <!--<mesh filename="package://realsense2_description/meshes/d435/d435.dae" />-->
       </geometry>
       <material name="camera_aluminum"/>
-    </visual>
+    </visual> -->
     <collision>
       <origin rpy="0 0 0" xyz="0 -0.0175 0"/>
@@ -793,4 +787,12 @@
   </link>
   <link name="table">
+    <contact>
+      <friction_anchor/>
+      <lateral_friction value="1"/>
+      <spinning_friction value="0.1"/>
+      <rolling_friction value="0.1"/>
+      <contact_cfm value="0.5"/>
+      <contact_erp value="1.0"/>
+    </contact>
     <visual>
       <geometry>
@@ -867,5 +869,5 @@
   <link name="camera_bottom_screw_frame"/>
   <joint name="camera_link_joint" type="fixed">
-    <origin rpy="0 0 0" xyz="0 0.0175 0.0125"/>
+    <origin rpy="0 0.4 0" xyz="0 0.0175 0.0125"/>
     <!-- <origin rpy="0.0 -0.0 0.0" xyz="-0.0 -0.0 -0.0"/> -->
     <parent link="camera_bottom_screw_frame"/>
@@ -887,5 +889,5 @@
     <parent link="world"/>
     <child link="camera_link_frontal"/>
-    <origin xyz="0.05 0.95 1.05" rpy="0.0 0.0 -1.57"/>
+    <origin xyz="0.05 0.95 1.05" rpy="0.0 0.3 -1.57"/>
   </joint>
   <joint name="camera_side_world" type="fixed">

File: ros_ws/src/ur5_rl/urdf/002_master_chef_can/model.urdf (robot description, URDF)
Before this commit: robot model.urdf, 2 links, 1 joints
Links:
- removed link dummy
- link objectLink: mass 0.2 -> 0.5
Joints:
- removed joint dummyJoint
